File: LDO.kicad_pcb (KiCad board)
At the start: 2 copper layers, 40 x 40 mm, 27 parts, among them J1 Stack_2x05, J2 VOUT, J3 VOUT, U1 LT3042xMSE, U2 DAC60502, U3 INA226

Commit message: Drop screw terminal, fix silkscreen, add LCSC parts and BOM
- Remove J2 screw terminal (13.8 mm, too tall for the stack); J3 header is the output
- Silkscreen labels 1.0 mm / 0.15 mm, add LDO v0.1 and DAC address labels
- MPN and LCSC fields on every orderable part, matched in schematic and PCB
- LDO_BOM.csv exported from the schematic
Parts:
- removed J2: VOUT, TerminalBlock_Phoenix:TerminalBlock_Phoenix_MKDS-1,5-2-5.08_1x02_P5.08mm_Horizontal
Routing:
- net /VOUT: track 24.8 -> 24.1 mm
Other:
- board text added: "48"
- board text added: "49"
- board text added: "4A"
- board text added: "4B"
- board text added: "DAC 0x"
- board text added: "LDO v0.1"
- board text removed: "0x48"
- board text removed: "0x49"
- board text removed: "0x4A"
- board text removed: "0x4B"

Commit message: Center J3 on the right edge and add v0.1 fabrication files
- J3 pins straddle the board's 20 mm midline; VOUT rerouted with 0.5 mm, 45-degree trace
- Gerbers and Excellon drills for JLCPCB (2 layers, 40x40 mm) zipped under fabrication/
Parts:
- moved J3 6.23 mm to (134.5, 118.7)
Routing:
- net /VOUT: track 24.1 -> 17.3 mm
Changed lines of the file:
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@@
 	(footprint "Connector_PinHeader_2.54mm:PinHeader_1x02_P2.54mm_Horizontal"
 		(layer "F.Cu")
-		(at 134.5 112.5)
+		(at 134.5 118.73)
 		(descr "Through hole angled pin header, 1x02, 2.54mm pitch, 6mm pin length, single row")
 		(tags "Through hole angled pin header THT 1x02 2.54mm single row")
@@
 	)
 	(segment
-		(start 132 115)
-		(end 134.5 112.5)
-		(width 0.5)
-		(layer "F.Cu")
-		(net "/VOUT")
-	)
-	(segment
-		(start 132 125.05)
-		(end 132 115)
-		(width 0.5)
-		(layer "F.Cu")
-		(net "/VOUT")
-	)
-	(segment
-		(start 132 125.05)
-		(end 131.5 125.55)
+		(start 134 118.73)
+		(end 134.5 118.73)
 		(width 0.5)
 		(layer "F.Cu")
@@
 	)
 	(segment
+		(start 125.5 125.55)
+		(end 130 125.55)
+		(width 0.5)
+		(layer "F.Cu")
+		(net "/VOUT")
+	)
+	(segment
+		(start 130 125.55)
+		(end 132 123.55)
+		(width 0.5)
+		(layer "F.Cu")
+		(net "/VOUT")
+	)
+	(segment
 		(start 125 125)
 		(end 124 124)
@@
 	)
 	(segment
-		(start 125.5 125.55)
-		(end 131.5 125.55)
+		(start 132 123.55)
+		(end 132 120.73)
 		(width 0.5)
 		(layer "F.Cu")
+		(net "/VOUT")
+	)
+	(segment
+		(start 132 120.73)
+		(end 134 118.73)
+		(width 0.5)
+		(layer "F.Cu")
