File: LDO.kicad_sch (KiCad schematic)
At the start: 0 parts

Commit message: Draw LDO board schematic
One LT3042 channel set by a DAC60502 through an RC filter on SET,
read back by an INA226 across a 0.5 ohm shunt, with a 2x5 stacking
header and solder-jumper I2C address select.
Parts:
- added C1, C3: 47uF 10V, Capacitor_SMD:C_1206_3216Metric_Pad1.33x1.80mm_HandSolder, symbol Device:C
- added C2: 4.7uF 10V, Capacitor_SMD:C_0805_2012Metric_Pad1.18x1.45mm_HandSolder, symbol Device:C
- added C4: 10uF 10V, Capacitor_SMD:C_0805_2012Metric_Pad1.18x1.45mm_HandSolder, symbol Device:C
- added C5, C7: 100nF, Capacitor_SMD:C_0805_2012Metric_Pad1.18x1.45mm_HandSolder, symbol Device:C
- added C6, C8: 1uF, Capacitor_SMD:C_0805_2012Metric_Pad1.18x1.45mm_HandSolder, symbol Device:C
- added J1: Stack_2x05, Connector_PinSocket_2.54mm:PinSocket_2x05_P2.54mm_Vertical, symbol Connector_Generic:Conn_02x05_Odd_Even
- added J2: VOUT, TerminalBlock_Phoenix:TerminalBlock_Phoenix_MKDS-1,5-2-5.08_1x02_P5.08mm_Horizontal, symbol Connector:Screw_Terminal_01x02
- added JP1: DAC 0x49 / INA 0x41, Jumper:SolderJumper-2_P1.3mm_Open_RoundedPad1.0x1.5mm, symbol Jumper:SolderJumper_2_Open
- added JP2: DAC 0x4A / INA 0x42, Jumper:SolderJumper-2_P1.3mm_Open_RoundedPad1.0x1.5mm, symbol Jumper:SolderJumper_2_Open
- added JP3: DAC 0x4B / INA 0x43, Jumper:SolderJumper-2_P1.3mm_Open_RoundedPad1.0x1.5mm, symbol Jumper:SolderJumper_2_Open
- added JP4: DAC 0x48 / INA 0x40, Jumper:SolderJumper-2_P1.3mm_Open_RoundedPad1.0x1.5mm, symbol Jumper:SolderJumper_2_Open
- added R1: 4.7, Resistor_SMD:R_0805_2012Metric_Pad1.20x1.40mm_HandSolder, symbol Device:R
- added R2: 1k 0.1%, Resistor_SMD:R_0805_2012Metric_Pad1.20x1.40mm_HandSolder, symbol Device:R
- added R3: 1.5k, Resistor_SMD:R_0805_2012Metric_Pad1.20x1.40mm_HandSolder, symbol Device:R
- added R4: 0.5 1%, Resistor_SMD:R_1206_3216Metric_Pad1.30x1.75mm_HandSolder, symbol Device:R
- added U1: LT3042xMSE, Package_SO:MSOP-10-1EP_3x3mm_P0.5mm_EP1.68x1.88mm, symbol Regulator_Linear:LT3042xMSE
- added U2: DAC60502, Package_SON:Texas_DRX_WSON-10_2.5x2.5mm_P0.5mm, symbol Analog_DAC:DAC60502
- added U3: INA226, Package_SO:TSSOP-10_3x3mm_P0.5mm, symbol Sensor_Energy:INA226
Connections:
- new net: R3.1, U1.5 (ILIM)
- new net: C6.1, U2.10 (VREFIO)
- new net: R2.1, U2.2 (VOUTA)
- new net +3V3: C5.1, C7.1, C8.1, J1.3 (Pin_3), JP1.2 (B), U2.1 (VDD), U2.5 (SPI2C), U3.6 (VS)
- new net +5V: J1.1 (Pin_1), R1.1
- new net ADDR: JP1.1 (A), JP2.1 (A), JP3.1 (A), JP4.1 (A), U2.7 (~{SYNC}/A0), U3.2 (A0)
- new net GND: C1.2, C2.2, C3.2, C4.2, C5.2, C6.2, C7.2, C8.2, J1.10 (Pin_10), J1.2 (Pin_2), J1.4 (Pin_4), J1.6 (Pin_6), J1.8 (Pin_8), J1.9 (Pin_9), J2.2 (Pin_2), JP4.2 (B), R3.2, U1.11 (GND), U1.8 (GND), U2.3 (RSTSEL), U2.4 (AGND), U3.1 (A1), U3.7 (GND)
- new net LDO_OUT: C4.1, R4.1, U1.10 (OUT), U3.10 (Vin+)
- new net SCL: J1.7 (Pin_7), JP3.2 (B), U2.6 (SCLK/SCL), U3.5 (SCL)
- new net SDA: J1.5 (Pin_5), JP2.2 (B), U2.8 (SDIN/SDA), U3.4 (SDA)
- new net SET: C3.1, R2.2, U1.7 (SET)
- new net VIN_F: C1.1, C2.1, R1.2, U1.1 (IN), U1.2 (IN), U1.3 (EN/UV), U1.6 (PGFB)
- new net VOUT: J2.1 (Pin_1), R4.2, U1.9 (OUTS), U3.8 (Vbus), U3.9 (Vin-)
- no-connect marks 0 -> 3
Other:
- note added: "0.5 ohm shunt: 82 mV range = 164 mA, 5 uA steps."
- note added: "1 Stacking header"
- note added: "2 Input RC filter (fc ~ 720 Hz)"
- note added: "3 LT3042 regulator"
- note added: "4 Shunt and output"
- note added: "5 DAC60502 + SET-pin RC filter (fc ~ 3.4 Hz)"
- note added: "5V and 3.3V come from the XIAO board. I2C pull-ups live on the XIAO board."
- note added: "6 INA226 readback"
- note added: "7 I2C address (fit one jumper)"
- note added: "Drop is 0.47 V at 100 mA. Place C2 at the LT3042 IN pins."
- note added: "I2C mode (SPI2C high), powers up at 0 V (RSTSEL low). Firmware: REF-DIV = 1, gain = 2 for 0-2.5 V. VOUTB spare. C5, C8 at VDD. 100 uA SET current x R2 = ~0.1 V offset."
- note added: "INA226 reads across R4 (Kelvin taps at the pads)."
- note added: "PGFB, EN/UV tied to IN (power good unused). R3 sets current limit (~100 mA, check). OUTS senses VOUT after the shunt."
- title: (none) -> LDO board - BLE stackable low-noise supply

Commit message: Fix LT3042 connections per datasheet
- Tie OUTS to OUT at C4 so the shunt stays outside the regulation loop
- Set ILIM with 1k (125 mA*kohm scale factor, ~125 mA limit)
- Add R5 10k minimum load for stability below 1 V
Parts:
- added R5: 10k, Resistor_SMD:R_0805_2012Metric_Pad1.20x1.40mm_HandSolder, symbol Device:R
- C4: value 10uF 10V -> 10uF
- R3: value 1.5k -> 1k 1%
Connections:
- net GND: now also R5.2
- net LDO_OUT: now also U1.9 (OUTS), R5.1
- net VOUT: no longer U1.9 (OUTS)
Other:
- note added: "INA226 reads across R4 (Kelvin taps at the pads). R4 is outside the LT3042 loop: VOUT sags 0.5 mV/mA, which firmware trims via the DAC."
- note added: "PGFB, EN/UV tied to IN; PG floats (unused). R3: 125 mA*kohm / 1k = ~125 mA limit. OUTS Kelvin to C4 (10V X7R, ESR < 50 mohm). R5 = 10 uA min load below 1 V. Tie C3 and C4 grounds together; R3 to GND pin."
- note removed: "INA226 reads across R4 (Kelvin taps at the pads)."
- note removed: "PGFB, EN/UV tied to IN (power good unused). R3 sets current limit (~100 mA, check). OUTS senses VOUT after the shunt."
Changed lines of the file:
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@@
 			)
 		)
-		(property "Value" "1.5k"
+		(property "Value" "1k 1%"
 			(at 154.94 58.42 0)
 			(effects
@@
 		)
 	)
-	(label "VOUT"
-		(at 185.42 48.26 0)
-		(effects
-			(font
-				(size 1.27 1.27)
-			)
-			(justify left bottom)
+	(wire
+		(pts
+			(xy 185.42 48.26)
+			(xy 185.42 45.72)
+		)
+		(stroke
+			(width 0)
+			(type default)
 		)
 	)
+	(junction
+		(at 185.42 45.72)
+		(diameter 0)
+		(color 0 0 0 0)
+	)
 	(symbol
 		(lib_id "Device:C")
@@
 			)
 		)
-		(property "Value" "10uF 10V"
+		(property "Value" "10uF"
 			(at 200.66 50.8 0)
 			(effects
@@
 		)
 	)
+	(symbol
+		(lib_id "Device:R")
+		(at 208.28 49.53 0)
+		(unit 1)
+		(exclude_from_sim no)
+		(in_bom yes)
+		(on_board yes)
+		(dnp no)
+		(property "Reference" "R5"
+			(at 210.82 48.26 0)
+			(effects
+				(font
+					(size 1.27 1.27)
+				)
+				(justify left)
+			)
+		)
+		(property "Value" "10k"
+			(at 210.82 50.8 0)
+			(effects
+				(font
+					(size 1.27 1.27)
+				)
+				(justify left)
+			)
+		)
+		(property "Footprint" "Resistor_SMD:R_0805_2012Metric_Pad1.20x1.40mm_HandSolder"
+			(at 208.28 49.53 0)
+			(effects
+				(font
+					(size 1.27 1.27)
+				)
+				(hide yes)
+			)
+		)
+		(property "Datasheet" ""
+			(at 208.28 49.53 0)
+			(effects
+				(font
+					(size 1.27 1.27)
+				)
+				(hide yes)
+			)
+		)
+		(property "Description" "Resistor"
+			(at 208.28 49.53 0)
+			(effects
+				(font
+					(size 1.27 1.27)
+				)
+				(hide yes)
+			)
+		)
+		(pin "1"
+		)
+		(pin "2"
+		)
+		(instances
+			(project "LDO"
+				(path "/9b6db749-0574-4f27-8407-d33b6417d2e0"
+					(reference "R5")
+					(unit 1)
+				)
+			)
+		)
+	)
 	(wire
 		(pts
 			(xy 182.88 45.72)
-			(xy 205.74 45.72)
+			(xy 213.36 45.72)
 		)
 		(stroke
@@
 		(color 0 0 0 0)
 	)
+	(junction
+		(at 208.28 45.72)
+		(diameter 0)
+		(color 0 0 0 0)
+	)
 	(symbol
 		(lib_id "power:GND")
@@
 		)
 	)
+	(symbol
+		(lib_id "power:GND")
+		(at 208.28 53.34 0)
+		(unit 1)
+		(exclude_from_sim no)
+		(in_bom no)
+		(on_board yes)
+		(dnp no)
+		(property "Reference" "#PWR014"
+			(at 208.28 59.69 0)
+			(effects
+				(font
+					(size 1.27 1.27)
+				)
+				(hide yes)
+			)
+		)
+		(property "Value" "GND"
+			(at 208.28 57.15 0)
+			(effects
+				(font
+					(size 1.27 1.27)
+				)
+			)
+		)
+		(property "Footprint" ""
+			(at 208.28 53.34 0)
+			(effects
+				(font
+					(size 1.27 1.27)
+				)
+				(hide yes)
+			)
+		)
+		(property "Datasheet" ""
+			(at 208.28 53.34 0)
+			(effects
+				(font
+					(size 1.27 1.27)
+				)
+				(hide yes)
+			)
+		)
+		(property "Description" "Power symbol creates a global label with name \"GND\" , ground"
+			(at 208.28 53.34 0)
+			(effects
+				(font
+					(size 1.27 1.27)
+				)
+				(hide yes)
+			)
+		)
+		(pin "1"
+		)
+		(instances
+			(project "LDO"
+				(path "/9b6db749-0574-4f27-8407-d33b6417d2e0"
+					(reference "#PWR014")
+					(unit 1)
+				)
+			)
+		)
+	)
 	(label "LDO_OUT"
-		(at 205.74 45.72 0)
+		(at 213.36 45.72 0)
 		(effects
 			(font
@@
 		)
 	)
-	(text "PGFB, EN/UV tied to IN (power good unused).\nR3 sets current limit (~100 mA, check).\nOUTS senses VOUT after the shunt."
+	(text "PGFB, EN/UV tied to IN; PG floats (unused).\nR3: 125 mA*kohm / 1k = ~125 mA limit.\nOUTS Kelvin to C4 (10V X7R, ESR < 50 mohm).\nR5 = 10 uA min load below 1 V.\nTie C3 and C4 grounds together; R3 to GND pin."
 		(exclude_from_sim no)
-		(at 142.24 78.74 0)
+		(at 142.24 76.2 0)
 		(effects
 			(font
@@
 		(on_board yes)
 		(dnp no)
-		(property "Reference" "#PWR014"
+		(property "Reference" "#PWR015"
 			(at 261.62 57.15 0)
 			(effects
@@
 			(project "LDO"
 				(path "/9b6db749-0574-4f27-8407-d33b6417d2e0"
-					(reference "#PWR014")
+					(reference "#PWR015")
 					(unit 1)
 				)
@@
 		)
 	)
-	(text "INA226 reads across R4\n(Kelvin taps at the pads)."
+	(text "INA226 reads across R4\n(Kelvin taps at the pads).\nR4 is outside the LT3042 loop:\nVOUT sags 0.5 mV/mA, which\nfirmware trims via the DAC."
 		(exclude_from_sim no)
-		(at 228.6 71.12 0)
+		(at 228.6 68.58 0)
 		(effects
 			(font
@@
 		(on_board yes)
 		(dnp no)
-		(property "Reference" "#PWR015"
+		(property "Reference" "#PWR016"
 			(at 58.42 113.03 0)
 			(effects
@@
 			(project "LDO"
 				(path "/9b6db749-0574-4f27-8407-d33b6417d2e0"
-					(reference "#PWR015")
+					(reference "#PWR016")
 					(unit 1)
 				)
@@
 		(on_board yes)
 		(dnp no)
-		(property "Reference" "#PWR016"
+		(property "Reference" "#PWR017"
 			(at 58.42 148.59 0)
 			(effects
@@
 			(project "LDO"
 				(path "/9b6db749-0574-4f27-8407-d33b6417d2e0"
-					(reference "#PWR016")
+					(reference "#PWR017")
 					(unit 1)
 				)
@@
 		(on_board yes)
 		(dnp no)
-		(property "Reference" "#PWR017"
+		(property "Reference" "#PWR018"
 			(at 43.18 120.65 0)
 			(effects
@@
 			(project "LDO"
 				(path "/9b6db749-0574-4f27-8407-d33b6417d2e0"
-					(reference "#PWR017")
+					(reference "#PWR018")
 					(unit 1)
 				)
@@
 		(on_board yes)
 		(dnp no)
-		(property "Reference" "#PWR018"
+		(property "Reference" "#PWR019"
 			(at 33.02 130.81 0)
 			(effects
@@
 			(project "LDO"
 				(path "/9b6db749-0574-4f27-8407-d33b6417d2e0"
-					(reference "#PWR018")
+					(reference "#PWR019")
 					(unit 1)
 				)
@@
 		(on_board yes)
 		(dnp no)
-		(property "Reference" "#PWR019"
+		(property "Reference" "#PWR020"
 			(at 78.74 133.35 0)
 			(effects
@@
 			(project "LDO"
 				(path "/9b6db749-0574-4f27-8407-d33b6417d2e0"
-					(reference "#PWR019")
+					(reference "#PWR020")
 					(unit 1)
 				)
@@
 		(on_board yes)
 		(dnp no)
-		(property "Reference" "#PWR020"
+		(property "Reference" "#PWR021"
 			(at 96.52 151.13 0)
 			(effects
@@
 			(project "LDO"
 				(path "/9b6db749-0574-4f27-8407-d33b6417d2e0"
-					(reference "#PWR020")
+					(reference "#PWR021")
 					(unit 1)
 				)
@@
 		(on_board yes)
 		(dnp no)
-		(property "Reference" "#PWR021"
+		(property "Reference" "#PWR022"
 			(at 22.86 138.43 0)
 			(effects
@@
 			(project "LDO"
 				(path "/9b6db749-0574-4f27-8407-d33b6417d2e0"
-					(reference "#PWR021")
+					(reference "#PWR022")
 					(unit 1)
 				)
@@
 		(on_board yes)
 		(dnp no)
-		(property "Reference" "#PWR022"
+		(property "Reference" "#PWR023"
 			(at 22.86 153.67 0)
 			(effects
@@
 			(project "LDO"
 				(path "/9b6db749-0574-4f27-8407-d33b6417d2e0"
-					(reference "#PWR022")
+					(reference "#PWR023")
 					(unit 1)
 				)
@@
 		(on_board yes)
 		(dnp no)
-		(property "Reference" "#PWR023"
+		(property "Reference" "#PWR024"
 			(at 33.02 138.43 0)
 			(effects
@@
 			(project "LDO"
 				(path "/9b6db749-0574-4f27-8407-d33b6417d2e0"
-					(reference "#PWR023")
+					(reference "#PWR024")
 					(unit 1)
 				)
@@
 		(on_board yes)
 		(dnp no)
-		(property "Reference" "#PWR024"
+		(property "Reference" "#PWR025"
 			(at 33.02 153.67 0)
 			(effects
@@
 			(project "LDO"
 				(path "/9b6db749-0574-4f27-8407-d33b6417d2e0"
-					(reference "#PWR024")
+					(reference "#PWR025")
 					(unit 1)
 				)
@@
 		(on_board yes)
 		(dnp no)
-		(property "Reference" "#PWR025"
+		(property "Reference" "#PWR026"
 			(at 165.1 113.03 0)
 			(effects
@@
 			(project "LDO"
 				(path "/9b6db749-0574-4f27-8407-d33b6417d2e0"
-					(reference "#PWR025")
+					(reference "#PWR026")
 					(unit 1)
 				)
@@
 		(on_board yes)
 		(dnp no)
-		(property "Reference" "#PWR026"
+		(property "Reference" "#PWR027"
 			(at 165.1 146.05 0)
 			(effects
@@
 			(project "LDO"
 				(path "/9b6db749-0574-4f27-8407-d33b6417d2e0"
-					(reference "#PWR026")
+					(reference "#PWR027")
 					(unit 1)
 				)
@@
 		(on_board yes)
 		(dnp no)
-		(property "Reference" "#PWR027"
+		(property "Reference" "#PWR028"
 			(at 187.96 125.73 0)
 			(effects
@@
 			(project "LDO"
 				(path "/9b6db749-0574-4f27-8407-d33b6417d2e0"
-					(reference "#PWR027")
+					(reference "#PWR028")
 					(unit 1)
 				)
@@
 		(on_board yes)
 		(dnp no)
-		(property "Reference" "#PWR028"
+		(property "Reference" "#PWR029"
 			(at 195.58 139.7 0)
 			(effects
@@
 			(project "LDO"
 				(path "/9b6db749-0574-4f27-8407-d33b6417d2e0"
-					(reference "#PWR028")
+					(reference "#PWR029")
 					(unit 1)
 				)
@@
 		(on_board yes)
 		(dnp no)
-		(property "Reference" "#PWR029"
+		(property "Reference" "#PWR030"
 			(at 195.58 154.94 0)
 			(effects
@@
 			(project "LDO"
 				(path "/9b6db749-0574-4f27-8407-d33b6417d2e0"
-					(reference "#PWR029")
+					(reference "#PWR030")
 					(unit 1)
 				)
@@
 		(on_board yes)
 		(dnp no)
-		(property "Reference" "#PWR030"
+		(property "Reference" "#PWR031"
 			(at 233.68 113.03 0)
 			(effects
@@
 			(project "LDO"
 				(path "/9b6db749-0574-4f27-8407-d33b6417d2e0"
-					(reference "#PWR030")
+					(reference "#PWR031")
 					(unit 1)
 				)
@@
 		(on_board yes)
 		(dnp no)
-		(property "Reference" "#PWR031"
+		(property "Reference" "#PWR032"
 			(at 233.68 154.94 0)
 			(effects
@@
 			(project "LDO"
 				(path "/9b6db749-0574-4f27-8407-d33b6417d2e0"
-					(reference "#PWR031")
+					(reference "#PWR032")
 					(unit 1)
 				)

Commit message: Add second 5V header pin and right-angle output header
- J1 pin 2 now carries 5V (two 5V pins, five GND pins)
- J3: 2-pin 2.54 mm right-angle header in parallel with the screw terminal
Parts:
- added J3: VOUT, Connector_PinHeader_2.54mm:PinHeader_1x02_P2.54mm_Horizontal, symbol Connector_Generic:Conn_01x02
Connections:
- net +5V: now also J1.2 (Pin_2)
- net GND: now also J3.2 (Pin_2); no longer J1.2 (Pin_2)
- net VOUT: now also J3.1 (Pin_1)

Commit message: Place and route the LDO board
- 40x40 mm 2-layer board with M3 corner holes, J1 stacking header on the left edge
- Small passives moved to 0603; jumpers excluded from the BOM; stable symbol IDs
- Solid GND fill on both layers with thermal reliefs for hand and hot-plate soldering
- LT3042 routed per datasheet: OUTS Kelvin at C4, C3/C4 grounds tied, thermal vias
- INA226 Kelvin taps on the shunt, I2C/ADDR fan-out, 45-degree corners throughout
- Ignore KiCad .history/
Parts:
- C5, C6, C7, C8: footprint Capacitor_SMD:C_0805_2012Metric_Pad1.18x1.45mm_HandSolder -> Capacitor_SMD:C_0603_1608Metric_Pad1.08x0.95mm_HandSolder
- JP1, JP2, JP3, JP4: now left out of the parts list
- R2, R3, R5: footprint Resistor_SMD:R_0805_2012Metric_Pad1.20x1.40mm_HandSolder -> Resistor_SMD:R_0603_1608Metric_Pad0.98x0.95mm_HandSolder
Changed lines of the file:
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@@
 			)
 		)
-		(property "Footprint" "Resistor_SMD:R_0805_2012Metric_Pad1.20x1.40mm_HandSolder"
+		(property "Footprint" "Resistor_SMD:R_0603_1608Metric_Pad0.98x0.95mm_HandSolder"
 			(at 152.4 57.15 0)
 			(effects
@@
 			)
 		)
-		(property "Footprint" "Resistor_SMD:R_0805_2012Metric_Pad1.20x1.40mm_HandSolder"
+		(property "Footprint" "Resistor_SMD:R_0603_1608Metric_Pad0.98x0.95mm_HandSolder"
 			(at 208.28 49.53 0)
 			(effects
@@
 			)
 		)
-		(property "Footprint" "Capacitor_SMD:C_0805_2012Metric_Pad1.18x1.45mm_HandSolder"
+		(property "Footprint" "Capacitor_SMD:C_0603_1608Metric_Pad1.08x0.95mm_HandSolder"
 			(at 78.74 123.19 0)
 			(effects
@@
 			)
 		)
-		(property "Footprint" "Resistor_SMD:R_0805_2012Metric_Pad1.20x1.40mm_HandSolder"
+		(property "Footprint" "Resistor_SMD:R_0603_1608Metric_Pad0.98x0.95mm_HandSolder"
 			(at 83.82 134.62 270)
 			(effects
@@
 			)
 		)
-		(property "Footprint" "Capacitor_SMD:C_0805_2012Metric_Pad1.18x1.45mm_HandSolder"
+		(property "Footprint" "Capacitor_SMD:C_0603_1608Metric_Pad1.08x0.95mm_HandSolder"
 			(at 22.86 140.97 0)
 			(effects
@@
 			)
 		)
-		(property "Footprint" "Capacitor_SMD:C_0805_2012Metric_Pad1.18x1.45mm_HandSolder"
+		(property "Footprint" "Capacitor_SMD:C_0603_1608Metric_Pad1.08x0.95mm_HandSolder"
 			(at 33.02 140.97 0)
 			(effects
@@
 			)
 		)
-		(property "Footprint" "Capacitor_SMD:C_0805_2012Metric_Pad1.18x1.45mm_HandSolder"
+		(property "Footprint" "Capacitor_SMD:C_0603_1608Metric_Pad1.08x0.95mm_HandSolder"
 			(at 195.58 142.24 0)
 			(effects
@@
 		(unit 1)
 		(exclude_from_sim no)
-		(in_bom yes)
+		(in_bom no)
 		(on_board yes)
 		(dnp no)
@@
 		(unit 1)
 		(exclude_from_sim no)
-		(in_bom yes)
+		(in_bom no)
 		(on_board yes)
 		(dnp no)
@@
 		(unit 1)
 		(exclude_from_sim no)
-		(in_bom yes)
+		(in_bom no)
 		(on_board yes)
 		(dnp no)
@@
 		(unit 1)
 		(exclude_from_sim no)
-		(in_bom yes)
+		(in_bom no)
 		(on_board yes)
 		(dnp no)

Commit message: Drop screw terminal, fix silkscreen, add LCSC parts and BOM
- Remove J2 screw terminal (13.8 mm, too tall for the stack); J3 header is the output
- Silkscreen labels 1.0 mm / 0.15 mm, add LDO v0.1 and DAC address labels
- MPN and LCSC fields on every orderable part, matched in schematic and PCB
- LDO_BOM.csv exported from the schematic
Parts:
- removed J2: VOUT, TerminalBlock_Phoenix:TerminalBlock_Phoenix_MKDS-1,5-2-5.08_1x02_P5.08mm_Horizontal, symbol Connector:Screw_Terminal_01x02
- C1, C3: LCSC (none) -> C96123; MPN (none) -> CL31A476MPHNNNE
- C2: LCSC (none) -> C98195; MPN (none) -> CL21B475KAFNNNE
- C4: LCSC (none) -> C15850; MPN (none) -> CL21A106KAYNNNE
- C5, C7: LCSC (none) -> C1591; MPN (none) -> CL10B104KB8NNNC
- C6, C8: LCSC (none) -> C29936; MPN (none) -> CL10B105KA8NNNC
- J1: LCSC (none) -> C22073008; MPN (none) -> ESW-105-12-L-D
- J3: LCSC (none) -> C492410; MPN (none) -> PZ254R-11-02P
- R1: LCSC (none) -> C137513; MPN (none) -> RC0805FR-074R7L
- R2: LCSC (none) -> C110776; MPN (none) -> RT0603BRD071KL
- R3: LCSC (none) -> C21190; MPN (none) -> 0603WAF1001T5E
- R4: LCSC (none) -> C327075; MPN (none) -> RL1206FR-070R5L
- R5: LCSC (none) -> C25804; MPN (none) -> 0603WAF1002T5E
- U1: LCSC (none) -> C69847; MPN (none) -> LT3042EMSE#PBF
- U2: LCSC (none) -> C2876322; MPN (none) -> DAC60502DRXR
- U3: LCSC (none) -> C49851; MPN (none) -> INA226AIDGSR
Other:
- moved on the sheet: J3

Commit message: Switch R1 to an in-stock part and drop J1's LCSC number
- R1: Yageo SR0805FR-7W4R7L (LCSC C873778, 250 mW); C137513 was out of stock
- J1: remove MPN/LCSC; the long-pin stacking socket is sourced separately
Parts:
- J1: LCSC C22073008 -> (none); MPN ESW-105-12-L-D -> (none)
- R1: LCSC C137513 -> C873778; MPN RC0805FR-074R7L -> SR0805FR-7W4R7L
Changed lines of the file:
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@@
-			)
-		)
-		(property "MPN" "ESW-105-12-L-D"
-			(at 35.56 48.26 0)
-			(effects
-				(font
-					(size 1.27 1.27)
-				)
-				(hide yes)
-			)
-		)
-		(property "LCSC" "C22073008"
-			(at 35.56 48.26 0)
-			(effects
-				(font
-					(size 1.27 1.27)
-				)
-				(hide yes)
 			)
 		)
@@
 			)
 		)
-		(property "MPN" "RC0805FR-074R7L"
+		(property "MPN" "SR0805FR-7W4R7L"
 			(at 83.82 45.72 270)
 			(effects
@@
 			)
 		)
-		(property "LCSC" "C137513"
+		(property "LCSC" "C873778"
 			(at 83.82 45.72 270)
 			(effects
