File: controller/controller.kicad_pcb (KiCad board)
At the start: 2 copper layers, 40 x 40 mm, 5 parts, among them J1 Stack_2x05

Commit message: Draw, place and route the controller board
Add a project-local XIAO nRF52840 symbol and castellated footprint, the
500 mA PTC fuse, 10 uF bulk cap and 4.7k I2C pull-ups. The XIAO sits at
the top edge with USB-C overhanging and a copper keepout under its
antenna. Add the BOM with LCSC numbers and the v0.1 Gerber zip.
Parts:
- added C1: 10uF 25V, Capacitor_SMD:C_0805_2012Metric_Pad1.18x1.45mm_HandSolder, F.Cu at (108.0, 129.0)
- added F1: 500mA, Fuse:Fuse_1206_3216Metric_Pad1.42x1.75mm_HandSolder, F.Cu at (133.2, 110.5)
- added R1: 4.7k, Resistor_SMD:R_0603_1608Metric_Pad0.98x0.95mm_HandSolder, F.Cu at (109.6, 110.6)
- added R2: 4.7k, Resistor_SMD:R_0603_1608Metric_Pad0.98x0.95mm_HandSolder, F.Cu at (109.2, 118.0)
- added U1: XIAO_nRF52840, controller:XIAO_nRF52840_SMD, F.Cu at (121.0, 110.5)
Routing:
- net +5V: track 0.00 -> 62.4 mm
- net +3V3: track 0.00 -> 41.0 mm, vias 0 -> 3
- net /SDA: track 0.00 -> 14.4 mm
- net /SCL: track 0.00 -> 13.8 mm
- net /VBUS: track 0.00 -> 9.13 mm
- net GND: track 0.00 -> 3.70 mm, vias 0 -> 11
- added copper zone on B.Cu, net GND
- added copper zone on F.Cu, net GND
Other:
- board text added: "CTRL v0.1"
