File: controller/controller.kicad_sch (KiCad schematic)
At the start: 1 part, among them J1 Stack_2x05

Commit message: Draw, place and route the controller board
Add a project-local XIAO nRF52840 symbol and castellated footprint, the
500 mA PTC fuse, 10 uF bulk cap and 4.7k I2C pull-ups. The XIAO sits at
the top edge with USB-C overhanging and a copper keepout under its
antenna. Add the BOM with LCSC numbers and the v0.1 Gerber zip.
Parts:
- added C1: 10uF 25V, Capacitor_SMD:C_0805_2012Metric_Pad1.18x1.45mm_HandSolder, symbol Device:C
- added F1: 500mA, Fuse:Fuse_1206_3216Metric_Pad1.42x1.75mm_HandSolder, symbol Device:Polyfuse
- added R1, R2: 4.7k, Resistor_SMD:R_0603_1608Metric_Pad0.98x0.95mm_HandSolder, symbol Device:R
- added U1: XIAO_nRF52840, controller:XIAO_nRF52840_SMD, symbol controller:XIAO_nRF52840
- J1: LCSC (none) -> C492399; MPN (none) -> PM254V-12-10P-H85
Connections:
- net +3V3: now also R1.1, R2.1, U1.12 (3V3)
- net +5V: now also C1.1, F1.2
- net GND: now also C1.2, U1.13 (GND)
- net SCL: now also R2.2, U1.6 (D5/SCL)
- net SDA: now also R1.2, U1.5 (D4/SDA)
- new net VBUS: F1.1, U1.14 (5V)
- no-connect marks 0 -> 9
Other:
- note added: "2 XIAO nRF52840 (soldered flat)"
- note added: "3 5V fuse and bulk capacitor"
- note added: "4 I2C pull-ups (only ones on the bus)"
- note added: "PTC fuse: 500 mA hold, 1 A trip. Limits a short on the stack instead of loading the XIAO and the USB port."
- note added: "The LDO boards have no pull-ups, so the bus has exactly these two."
- note added: "USB-C at the board edge powers everything. 5V pin = USB VBUS (to the fuse); 3V3 pin feeds the DACs and INA226s on the LDO boards (a few mA). Keep copper away from the antenna end."
